Commit message: fix(urdf): add dummy finger_joint1 to URDF to prevent joint_state_broadcaster array mismatch

File: src/panda_mjk/urdf/panda.urdf.xacro (robot description, xacro)
@@ -32,4 +32,17 @@
                       tcp_rpy="0 0 0"
                       no_prefix="false" />
+  <!-- Dummy link and joint for finger_joint1 to satisfy joint_state_broadcaster.
+       Because hand="false" is set above, the hand links aren't generated. However,
+       we still export finger_joint1 in ros2_control for the gripper action server.
+       If the joint doesn't exist in the URDF, joint_state_broadcaster pushes its
+       position but skips its name, leading to an array size mismatch crash. -->
+  <link name="fer_leftfinger_dummy"/>
+  <joint name="finger_joint1" type="prismatic">
+    <parent link="fer_link7"/>
+    <child link="fer_leftfinger_dummy"/>
+    <origin xyz="0 0 0.1654" rpy="0 0 0"/>
+    <axis xyz="0 1 0"/>
+    <limit lower="0.0" upper="0.04" effort="100" velocity="0.2"/>
+  </joint>
   <!-- ros2_control definition -->
   <ros2_control name="FrankaSystem" type="system">

Commit message: fix(urdf): add dummy finger_joint2 to URDF to fix position=9 array mismatch

File: src/panda_mjk/urdf/panda.urdf.xacro (robot description, xacro)
@@ -43,4 +43,12 @@
     <origin xyz="0 0 0.1654" rpy="0 0 0"/>
     <axis xyz="0 1 0"/>
+    <limit lower="0.0" upper="0.04" effort="100" velocity="0.2"/>
+  </joint>
+  <link name="fer_rightfinger_dummy"/>
+  <joint name="finger_joint2" type="prismatic">
+    <parent link="fer_link7"/>
+    <child link="fer_rightfinger_dummy"/>
+    <origin xyz="0 0 0.1654" rpy="0 0 0"/>
+    <axis xyz="0 -1 0"/>
     <limit lower="0.0" upper="0.04" effort="100" velocity="0.2"/>
   </joint>

Commit message: fix(controllers): configure explicit joints/interfaces for joint_state_broadcaster and remove dummy finger_joint2

File: src/panda_mjk/urdf/panda.urdf.xacro (robot description, xacro)
@@ -32,9 +32,7 @@
                       tcp_rpy="0 0 0"
                       no_prefix="false" />
-  <!-- Dummy link and joint for finger_joint1 to satisfy joint_state_broadcaster.
-       Because hand="false" is set above, the hand links aren't generated. However,
-       we still export finger_joint1 in ros2_control for the gripper action server.
-       If the joint doesn't exist in the URDF, joint_state_broadcaster pushes its
-       position but skips its name, leading to an array size mismatch crash. -->
+  <!-- Dummy link and joint for finger_joint1.
+       Because hand="false" is set above, the hand links aren't generated from franka_description.
+       We define finger_joint1 here for TF/kinematics corresponding to the gripper joint. -->
   <link name="fer_leftfinger_dummy"/>
   <joint name="finger_joint1" type="prismatic">
@@ -43,12 +41,4 @@
     <origin xyz="0 0 0.1654" rpy="0 0 0"/>
     <axis xyz="0 1 0"/>
-    <limit lower="0.0" upper="0.04" effort="100" velocity="0.2"/>
-  </joint>
-  <link name="fer_rightfinger_dummy"/>
-  <joint name="finger_joint2" type="prismatic">
-    <parent link="fer_link7"/>
-    <child link="fer_rightfinger_dummy"/>
-    <origin xyz="0 0 0.1654" rpy="0 0 0"/>
-    <axis xyz="0 -1 0"/>
     <limit lower="0.0" upper="0.04" effort="100" velocity="0.2"/>
   </joint>
@@ -105,4 +95,5 @@
         <param name="initial_value">0.0</param>
       </state_interface>
+      <state_interface name="effort"/>
     </joint>
     <!-- On real hardware, franka_hardware exposes nothing for gripper. On sim, mujoco_ros2_control can. -->

Commit message: fix: unify 9-joint set (fer_joint1-7 + finger_joint1-2) across URDF, ros2_control, and controllers.yaml

File: src/panda_mjk/urdf/panda.urdf.xacro (robot description, xacro)
@@ -32,7 +32,7 @@
                       tcp_rpy="0 0 0"
                       no_prefix="false" />
-  <!-- Dummy link and joint for finger_joint1.
+  <!-- Dummy links and joints for gripper fingers.
        Because hand="false" is set above, the hand links aren't generated from franka_description.
-       We define finger_joint1 here for TF/kinematics corresponding to the gripper joint. -->
+       We define finger_joint1 and finger_joint2 here for TF/kinematics corresponding to the gripper joints. -->
   <link name="fer_leftfinger_dummy"/>
   <joint name="finger_joint1" type="prismatic">
@@ -41,4 +41,12 @@
     <origin xyz="0 0 0.1654" rpy="0 0 0"/>
     <axis xyz="0 1 0"/>
+    <limit lower="0.0" upper="0.04" effort="100" velocity="0.2"/>
+  </joint>
+  <link name="fer_rightfinger_dummy"/>
+  <joint name="finger_joint2" type="prismatic">
+    <parent link="fer_link7"/>
+    <child link="fer_rightfinger_dummy"/>
+    <origin xyz="0 0 0.1654" rpy="0 0 0"/>
+    <axis xyz="0 -1 0"/>
     <limit lower="0.0" upper="0.04" effort="100" velocity="0.2"/>
   </joint>
@@ -86,7 +94,16 @@
     <xacro:configure_joint joint_name="fer_joint6"/>
     <xacro:configure_joint joint_name="fer_joint7"/>
-    <!-- Gripper joint definition (Only finger_joint1 is needed as control interface, finger_joint2 is mimicked/coupled) -->
+    <!-- Gripper joint definition (finger_joint1 has command+state, finger_joint2 has state exported from sim) -->
     <joint name="finger_joint1">
       <command_interface name="position" />
+      <state_interface name="position">
+        <param name="initial_value">0.0</param>
+      </state_interface>
+      <state_interface name="velocity">
+        <param name="initial_value">0.0</param>
+      </state_interface>
+      <state_interface name="effort"/>
+    </joint>
+    <joint name="finger_joint2">
       <state_interface name="position">
         <param name="initial_value">0.0</param>

Commit message: fix(launch): pass --param-file controllers_config to spawners and lock joint_state_broadcaster to 8 declared joints

File: src/panda_mjk/urdf/panda.urdf.xacro (robot description, xacro)
@@ -32,7 +32,7 @@
                       tcp_rpy="0 0 0"
                       no_prefix="false" />
-  <!-- Dummy links and joints for gripper fingers.
+  <!-- Dummy link and joint for finger_joint1.
        Because hand="false" is set above, the hand links aren't generated from franka_description.
-       We define finger_joint1 and finger_joint2 here for TF/kinematics corresponding to the gripper joints. -->
+       We define finger_joint1 here for TF/kinematics corresponding to the gripper joint. -->
   <link name="fer_leftfinger_dummy"/>
   <joint name="finger_joint1" type="prismatic">
@@ -41,12 +41,4 @@
     <origin xyz="0 0 0.1654" rpy="0 0 0"/>
     <axis xyz="0 1 0"/>
-    <limit lower="0.0" upper="0.04" effort="100" velocity="0.2"/>
-  </joint>
-  <link name="fer_rightfinger_dummy"/>
-  <joint name="finger_joint2" type="prismatic">
-    <parent link="fer_link7"/>
-    <child link="fer_rightfinger_dummy"/>
-    <origin xyz="0 0 0.1654" rpy="0 0 0"/>
-    <axis xyz="0 -1 0"/>
     <limit lower="0.0" upper="0.04" effort="100" velocity="0.2"/>
   </joint>
@@ -94,16 +86,7 @@
     <xacro:configure_joint joint_name="fer_joint6"/>
     <xacro:configure_joint joint_name="fer_joint7"/>
-    <!-- Gripper joint definition (finger_joint1 has command+state, finger_joint2 has state exported from sim) -->
+    <!-- Gripper joint definition (Only finger_joint1 is needed as control interface, finger_joint2 is mimicked/coupled in physics) -->
     <joint name="finger_joint1">
       <command_interface name="position" />
-      <state_interface name="position">
-        <param name="initial_value">0.0</param>
-      </state_interface>
-      <state_interface name="velocity">
-        <param name="initial_value">0.0</param>
-      </state_interface>
-      <state_interface name="effort"/>
-    </joint>
-    <joint name="finger_joint2">
       <state_interface name="position">
         <param name="initial_value">0.0</param>

Commit message: fix(robot_description): synchronize finger_joint2 across URDF, ros2_control, controllers.yaml, and dashboard

File: src/panda_mjk/urdf/panda.urdf.xacro (robot description, xacro)
@@ -32,7 +32,7 @@
                       tcp_rpy="0 0 0"
                       no_prefix="false" />
-  <!-- Dummy link and joint for finger_joint1.
+  <!-- Dummy links and joints for finger_joint1 and finger_joint2.
        Because hand="false" is set above, the hand links aren't generated from franka_description.
-       We define finger_joint1 here for TF/kinematics corresponding to the gripper joint. -->
+       We define finger_joint1 and finger_joint2 here for TF/kinematics corresponding to the gripper joints. -->
   <link name="fer_leftfinger_dummy"/>
   <joint name="finger_joint1" type="prismatic">
@@ -42,4 +42,13 @@
     <axis xyz="0 1 0"/>
     <limit lower="0.0" upper="0.04" effort="100" velocity="0.2"/>
+  </joint>
+  <link name="fer_rightfinger_dummy"/>
+  <joint name="finger_joint2" type="prismatic">
+    <parent link="fer_link7"/>
+    <child link="fer_rightfinger_dummy"/>
+    <origin xyz="0 0 0.1654" rpy="0 0 0"/>
+    <axis xyz="0 -1 0"/>
+    <limit lower="0.0" upper="0.04" effort="100" velocity="0.2"/>
+    <mimic joint="finger_joint1" multiplier="1.0" offset="0.0"/>
   </joint>
   <!-- ros2_control definition -->
@@ -86,7 +95,18 @@
     <xacro:configure_joint joint_name="fer_joint6"/>
     <xacro:configure_joint joint_name="fer_joint7"/>
-    <!-- Gripper joint definition (Only finger_joint1 is needed as control interface, finger_joint2 is mimicked/coupled in physics) -->
+    <!-- Gripper joint definitions -->
     <joint name="finger_joint1">
       <command_interface name="position" />
+      <state_interface name="position">
+        <param name="initial_value">0.0</param>
+      </state_interface>
+      <state_interface name="velocity">
+        <param name="initial_value">0.0</param>
+      </state_interface>
+      <state_interface name="effort"/>
+    </joint>
+    <joint name="finger_joint2">
+      <param name="mimic">finger_joint1</param>
+      <param name="multiplier">1.0</param>
       <state_interface name="position">
         <param name="initial_value">0.0</param>
